File: STM32DryerPCB_V2.kicad_pcb (KiCad board)
At the start: 2 copper layers, 100 x 100 mm, 100 parts, among them J1 AC_IN, J2 B1_B2_LCD, J3 B2_TEMP, J4 B2_INPUT, J5 B2_UART, J7 B3_output, J8 Conn_01x05, Q1 BD139, Q2 BD139, Q3 BD139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

Commit message: Fixed Boot pin not grounded
Parts:
- D5: value 1N5822 -> 1N5822/1N5819
- L1: value 68uH -> 470uH
- R2: value 1K -> 3.3K
- R3: value 1K -> 10K
Connections:
- U1 pad 44: unconnected-(U1-Pad44) -> GND
Routing:
- net GND: track 20.4 -> 21.9 mm, vias 33 -> 34
- net +3.3V: track 49.1 -> 48.1 mm
